File: pcb/barleycorn.sch (KiCad schematic (older format))
At the start: 223 parts, among them J1 USB4085-GF-A_REVA, J2 I2C, J3 ISP, SW1 SW_Push, SW10 SW_Push, SW11 SW_Push, SW12 SW_Push, SW13 SW_Push, SW14 SW_Push, SW15 SW_Push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

Commit message: Printed Schematic
Changed lines of the file:
@@
 Wire Wire Line
 	2775 3525 2875 3525
-Text Label -250 7675 0    50   ~ 10
-COL13
-Wire Wire Line
-	-350 7675 -250 7675
-Text Label -250 7775 0    50   ~ 10
-COL12
-Wire Wire Line
-	-350 7775 -250 7775
 NoConn ~ 2875 9325
 NoConn ~ 2875 9425
